File: hardware/hexaGenMini-v1/hexaGenMini-v1.kicad_sch (KiCad schematic)
At the start: 0 parts

Commit message: Add base schematic for hardware
Connections:
- no-connect marks 0 -> 17
Other:
- sheet CONNECTOR ports: added USB_DM, USB_DP, USB_VBUS_PIN; removed none
- sheet DDS ports: added DDS_CLKIN, DDS_D0, DDS_D1, DDS_D7, DDS_FQ_UD, DDS_IOUT, DDS_IOUTB, DDS_IOUTF, DDS_QOUT, DDS_QOUTB, DDS_RESET, DDS_VINP, DDS_W_CLK; removed none
- sheet MCU ports: added DDS_D7, DDS_FQ_UD, DDS_RESET, DDS_W_CLK, QSPI_SCLK, QSPI_SD0, QSPI_SD1, QSPI_SD2, QSPI_SD3, QSPI_SS, SWCLK, SWD, USB_DM, USB_DP, USB_VBUS_PIN; removed none

Commit message: Finish first hardware basic
Parts:
- added H1, H2, H3, H4: MountingHole, MountingHole:MountingHole_2.5mm, symbol Mechanical:MountingHole
Connections:
- no-connect marks 17 -> 0
Other:
- sheet CONNECTOR ports: added USB_DN; removed USB_DM
- sheet DDS ports: added none; removed DDS_CLKIN, DDS_D0, DDS_D1, DDS_IOUT, DDS_IOUTB, DDS_IOUTF, DDS_QOUT, DDS_QOUTB, DDS_VINP
- sheet MCU ports: added USB_DN; removed QSPI_SCLK, QSPI_SD0, QSPI_SD1, QSPI_SD2, QSPI_SD3, QSPI_SS, SWCLK, SWD, USB_DM
