File: hardware/hexaGenMini-v1/hexaGenMini-v1.kicad_pcb (KiCad board)
At the start: 2 copper layers, 0 parts

Commit message: Finish first hardware basic
Parts:
- added C1: 10uF, Capacitor_SMD:C_0805_2012Metric, F.Cu at (147.8, 105.8)
- added C10: 100nF, Capacitor_SMD:C_0402_1005Metric, F.Cu at (155.9, 100.2)
- added C11: 100nF, Capacitor_SMD:C_0402_1005Metric, F.Cu at (153.9, 95.9)
- added C12: 100nF, Capacitor_SMD:C_0402_1005Metric, F.Cu at (153.9, 94.9)
- added C13: 100nF, Capacitor_SMD:C_0402_1005Metric, F.Cu at (153.7, 93.4)
- added C14: 100nF, Capacitor_SMD:C_0402_1005Metric, F.Cu at (154.6, 93.4)
- added C15: 100nF, Capacitor_SMD:C_0402_1005Metric, F.Cu at (155.6, 93.4)
- added C16: 100nF, Capacitor_SMD:C_0402_1005Metric, F.Cu at (156.6, 93.4)
- added C17: 100nF, Capacitor_SMD:C_0402_1005Metric, F.Cu at (153.9, 96.8)
- added C18: 1uF, Capacitor_SMD:C_0603_1608Metric, F.Cu at (166.8, 102.7)
- added C19: 470pF, Capacitor_SMD:C_0402_1005Metric, F.Cu at (158.3, 77.1)
- added C2: 100nF, Capacitor_SMD:C_0402_1005Metric, F.Cu at (146.3, 105.0)
- added C20: 0.1uF, Capacitor_SMD:C_0402_1005Metric, F.Cu at (161.9, 61.2)
- added C21: 0.1uF, Capacitor_SMD:C_0402_1005Metric, F.Cu at (162.9, 61.2)
- added C22: 0.1uF, Capacitor_SMD:C_0402_1005Metric, F.Cu at (160.9, 61.2)
- added C23: 0.1uF, Capacitor_SMD:C_0402_1005Metric, F.Cu at (159.9, 61.2)
- added C24: 0.1uF, Capacitor_SMD:C_0402_1005Metric, F.Cu at (163.9, 61.2)
- added C25: 10uF Tantalum, Capacitor_Tantalum_SMD:CP_EIA-3216-18_Kemet-A, F.Cu at (166.8, 61.6)
- added C26: 22pF, Capacitor_SMD:C_0402_1005Metric, F.Cu at (154.4, 71.7)
- added C27: 33pF, Capacitor_SMD:C_0402_1005Metric, F.Cu at (152.1, 71.7)
- added C28: 22pF, Capacitor_SMD:C_0402_1005Metric, F.Cu at (149.7, 71.7)
- added C29: 22pF, Capacitor_SMD:C_0402_1005Metric, F.Cu at (147.3, 71.7)
- added C3: 100nF, Capacitor_SMD:C_0402_1005Metric, F.Cu at (151.0, 98.6)
- added C30: 1pF, Capacitor_SMD:C_0402_1005Metric, F.Cu at (153.9, 68.2)
- added C31: 5.6pF, Capacitor_SMD:C_0402_1005Metric, F.Cu at (150.9, 68.2)
- added C32: 4.7pF, Capacitor_SMD:C_0402_1005Metric, F.Cu at (147.9, 68.2)
- added C33: 470pF, Capacitor_SMD:C_0402_1005Metric, F.Cu at (157.3, 77.1)
- added C4: 10uF, Capacitor_SMD:C_0805_2012Metric, F.Cu at (151.8, 100.1)
- added C5: 27p, Capacitor_SMD:C_0402_1005Metric, F.Cu at (167.1, 89.2)
- added C6: 27p, Capacitor_SMD:C_0402_1005Metric, F.Cu at (169.7, 87.0)
- added C7: 1uF, Capacitor_SMD:C_0603_1608Metric, F.Cu at (155.3, 98.1)
- added C8: 1uF, Capacitor_SMD:C_0603_1608Metric, F.Cu at (156.3, 95.8)
- added C9: 100nF, Capacitor_SMD:C_0402_1005Metric, F.Cu at (155.9, 99.3)
- added D1: SMF5V0A, Diode_SMD:D_SMF, F.Cu at (151.1, 105.3)
- added D2: WS2812B, LED_SMD:LED_WS2812B_PLCC4_5.0x5.0mm_P3.2mm, F.Cu at (160.0, 84.0)
- added H1: MountingHole, MountingHole:MountingHole_2.5mm, F.Cu at (173.0, 61.5)
- added H2: MountingHole, MountingHole:MountingHole_2.5mm, F.Cu at (186.0, 84.0)
- added H3: MountingHole, MountingHole:MountingHole_2.5mm, F.Cu at (147.0, 61.5)
- added H4: MountingHole, MountingHole:MountingHole_2.5mm, F.Cu at (134.0, 84.0)
- added J1: Conn_Coaxial, Connector_Coaxial:SMA_Samtec_SMA-J-P-H-ST-EM1_EdgeMount, F.Cu at (179.7, 70.5)
- added J2: Conn_Coaxial, Connector_Coaxial:SMA_Samtec_SMA-J-P-H-ST-EM1_EdgeMount, F.Cu at (140.2, 70.5)
- added J3: Conn_01x03_Pin, Connector_PinHeader_2.54mm:PinHeader_1x03_P2.54mm_Vertical, F.Cu at (150.3, 83.8)
- added J4: USB_C_Receptacle_USB2.0_16P, Connector_USB:USB_C_Receptacle_HRO_TYPE-C-31-M-12, F.Cu at (160.0, 106.0)
- added L1: 470nH, Inductor_SMD:L_0603_1608Metric, F.Cu at (153.9, 70.5)
- added L2: 390nH, Inductor_SMD:L_0603_1608Metric, F.Cu at (150.9, 70.5)
- added L3: 390nH, Inductor_SMD:L_0603_1608Metric, F.Cu at (147.9, 70.5)
- added R1: 5.1k, Resistor_SMD:R_0603_1608Metric, F.Cu at (152.0, 107.2)
- added R10: 1k, Resistor_SMD:R_0603_1608Metric, F.Cu at (165.1, 65.1)
- added R11: 10k, Resistor_SMD:R_0603_1608Metric, F.Cu at (166.6, 65.1)
- added R12: 3.9k, Resistor_SMD:R_0603_1608Metric, F.Cu at (157.6, 65.1)
- added R13: 100, Resistor_SMD:R_0603_1608Metric, F.Cu at (159.5, 77.7)
- added R15: 100, Resistor_SMD:R_0603_1608Metric, F.Cu at (161.0, 77.7)
- added R16: 200, Resistor_SMD:R_0603_1608Metric, F.Cu at (156.1, 71.2)
- added R17: 200, Resistor_SMD:R_0603_1608Metric, F.Cu at (145.6, 71.2)
- added R19: 330, Resistor_SMD:R_0603_1608Metric, F.Cu at (165.0, 82.3)
- added R2: 5.1k, Resistor_SMD:R_0603_1608Metric, F.Cu at (152.0, 108.7)
- added R3: 5.6k, Resistor_SMD:R_0603_1608Metric, F.Cu at (152.0, 103.3)
- added R4: 10k, Resistor_SMD:R_0603_1608Metric, F.Cu at (152.0, 101.8)
- added R5: 1k, Resistor_SMD:R_0603_1608Metric, F.Cu at (167.1, 84.5)
- added R6: 27, Resistor_SMD:R_0603_1608Metric, F.Cu at (160.7, 97.4)
- added R7: 27, Resistor_SMD:R_0603_1608Metric, F.Cu at (159.2, 97.4)
- added R8: 10k, Resistor_SMD:R_0603_1608Metric, F.Cu at (169.8, 102.7)
- added R9: 1k, Resistor_SMD:R_0603_1608Metric, F.Cu at (172.8, 102.7)
- added SW1: SW_Push, Button_Switch_SMD:SW_SPST_B3U-1000P, F.Cu at (153.8, 84.4)
- added SW2: SW_Push, Button_Switch_SMD:SW_SPST_B3U-1000P, F.Cu at (171.9, 105.1)
- added U1: AMS1117-3.3, Package_TO_SOT_SMD:SOT-223-3_TabPin2, F.Cu at (144.6, 95.4)
- added U2: RP2040, Package_DFN_QFN:QFN-56-1EP_7x7mm_P0.4mm_EP3.2x3.2mm, F.Cu at (161.2, 91.8)
- added U3: AD9850, Package_SO:SSOP-28_5.3x10.2mm_P0.65mm, F.Cu at (162.4, 71.4)
- added U4: TPD2EUSB30, Package_TO_SOT_SMD:Texas_DRT-3, F.Cu at (160.0, 99.6)
- added U5: W25Q128JVS, Package_SO:SOIC-8_5.3x5.3mm_P1.27mm, F.Cu at (170.0, 99.0)
- added Y1: 12MHz 18pF, Crystal:Crystal_SMD_3225-4Pin_3.2x2.5mm, F.Cu at (167.1, 87.0)
- added Y2: XO53, Oscillator:Oscillator_SMD_EuroQuartz_XO53-4Pin_5.0x3.2mm, F.Cu at (161.4, 64.5)
Routing:
- net +5V: track 0.00 -> 94.7 mm, vias 0 -> 7
- net +3.3V: track 0.00 -> 69.6 mm, vias 0 -> 6
- net /DDS/DDS_W_CLK: track 0.00 -> 37.4 mm, vias 0 -> 2
- net /DDS/DDS_FQ_UD: track 0.00 -> 37.3 mm, vias 0 -> 2
- net /DDS/DDS_RESET: track 0.00 -> 28.7 mm
- net /CONNECTOR/USB_VBUS_PIN: track 0.00 -> 28.1 mm, vias 0 -> 2
- net /DDS/DDS_D7: track 0.00 -> 27.5 mm
- net Net-(J2-In): track 0.00 -> 26.9 mm
- net Net-(J1-In): track 0.00 -> 23.5 mm
- net /MCU/QSPI_SS: track 0.00 -> 23.3 mm
- net /MCU/RGB_LED: track 0.00 -> 20.9 mm
- net VBUS: track 0.00 -> 18.6 mm, vias 0 -> 3
- net /MCU/QSPI_SD1: track 0.00 -> 18.4 mm
- net +1V1: track 0.00 -> 17.5 mm
- net /MCU/SWD: track 0.00 -> 14.9 mm
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- added copper zone on B.Cu, net GND
- added copper zone on F.Cu, net GND
Other:
- board outline added: 58.5 x 52 mm
- board text added: "SINE OUT"
- board text added: "SQUARE OUT"
- board text added: "hexaGen Mini v1"

Commit message: Finish first hardware basic
Routing:
- net +5V: track 94.7 -> 95.2 mm
- net GND: vias 44 -> 115
Other:
- board text added: "BOOT"
- board text added: "GND"
- board text added: "RESET"
- board text added: "SWCLK"
- board text added: "SWD"
