File: hardware/hexaGenMini-v1/CONNECTOR.kicad_sch (KiCad schematic)
At the start: 7 parts, among them J1 USB_C_Receptacle, U4 TPD4E05U06DQA

Commit message: Add base schematic for hardware
Parts:
- J1: footprint (none) -> Connector_USB:USB_C_Receptacle_HRO_TYPE-C-31-M-12
- R1, R2, R3, R4: footprint (none) -> Capacitor_SMD:C_0603_1608Metric
Connections:
- net D+ renamed USB_DP
- net D- renamed USB_DM

Commit message: Finish first hardware basic
Parts:
- removed J1: USB_C_Receptacle, Connector_USB:USB_C_Receptacle_HRO_TYPE-C-31-M-12, symbol Connector:USB_C_Receptacle
- removed U4: TPD4E05U06DQA, Package_SON:USON-10_2.5x1.0mm_P0.5mm, symbol Power_Protection:TPD4E05U06DQA
- added J4: USB_C_Receptacle_USB2.0_16P, Connector_USB:USB_C_Receptacle_HRO_TYPE-C-31-M-12, symbol SCH_Library:USB_C_Receptacle_USB2.0_16P
- added U4: TPD2EUSB30, Package_TO_SOT_SMD:Texas_DRT-3, symbol Power_Protection:TPD2EUSB30
- D1: symbol Diode:SMF5V0A -> SCH_Library:SMF5V0A
- R1, R2, R3, R4: footprint Capacitor_SMD:C_0603_1608Metric -> Resistor_SMD:R_0603_1608Metric; symbol Device:R_Small -> SCH_Library:R_Small
Connections:
- net GND: now also J4.A1 (GND), J4.A12 (GND), J4.B1 (GND), J4.B12 (GND), J4.S1 (SHIELD), U4.3 (GND)
- net USB_DP: now also J4.A6 (D+), J4.B6 (D+), U4.1 (D+)
- net VBUS: now also J4.A4 (VBUS), J4.A9 (VBUS), J4.B4 (VBUS), J4.B9 (VBUS)
- net at R1.2: now also J4.A5 (CC1)
- net at R2.2: now also J4.B5 (CC2)
- new net USB_DN: J4.A7 (D-), J4.B7 (D-), U4.2 (D-)
- no-connect marks 10 -> 2

Commit message: Finish first hardware basic
Parts:
- D1: value SMF5V0A -> ESD DIODE 5VWM 9.2VC; LCSPN (none) -> C1972946; MFR (none) -> VISHAY; MPN (none) -> SMF5V0A-E3-08
- J4: LCSPN (none) -> C49261569; MFR (none) -> hanxia; MPN (none) -> HX-TYPE-C 16P 180 LT H10.0 USB 2.0 TYPE-C
- R1, R2: value 5.1k -> 5.1kΩ ±1% 100mW; LCSPN (none) -> C2907044; MFR (none) -> FOJAN; MPN (none) -> FRC0603F5101TS
- R3: value 5.6k -> 5.6kΩ ±1% 100mW; LCSPN (none) -> C2907046; MFR (none) -> FOJAN; MPN (none) -> FRC0603F5601TS
- R4: value 10k -> 10kΩ ±1% 100mW; LCSPN (none) -> C25804; MFR (none) -> UNI-ROYAL; MPN (none) -> 0603WAF1002T5E
- U4: value TPD2EUSB30 -> TVS DIODE 5.5VWM 18VC; LCSPN (none) -> C5182099; MFR (none) -> TECH PUBLIC; MPN (none) -> TPD2EUSB30DRTR
Changed lines of the file:
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@@
+			)
+		)
+		(property "MFR" "hanxia"
+			(at 111.76 68.58 0)
+			(effects
+				(font
+					(size 1.27 1.27)
+				)
+				(hide yes)
+			)
+		)
+		(property "MPN" "HX-TYPE-C 16P 180 LT H10.0 USB 2.0 TYPE-C"
+			(at 111.76 68.58 0)
+			(effects
+				(font
+					(size 1.27 1.27)
+				)
+				(hide yes)
+			)
+		)
+		(property "LCSPN" "C49261569"
+			(at 111.76 68.58 0)
+			(effects
+				(font
+					(size 1.27 1.27)
+				)
+				(hide yes)
 			)
 		)
@@
 			)
 		)
-		(property "Value" "TPD2EUSB30"
+		(property "Value" "TVS DIODE 5.5VWM 18VC"
 			(at 175.26 68.58 0)
 			(effects
@@
 		)
 		(property "Description" "2-Channel ESD Protection for Super-Speed USB 3.0 Interface, DRT-3"
+			(at 175.26 76.2 0)
+			(effects
+				(font
+					(size 1.27 1.27)
+				)
+				(hide yes)
+			)
+		)
+		(property "MFR" "TECH PUBLIC"
+			(at 175.26 76.2 0)
+			(effects
+				(font
+					(size 1.27 1.27)
+				)
+				(hide yes)
+			)
+		)
+		(property "MPN" "TPD2EUSB30DRTR"
+			(at 175.26 76.2 0)
+			(effects
+				(font
+					(size 1.27 1.27)
+				)
+				(hide yes)
+			)
+		)
+		(property "LCSPN" "C5182099"
 			(at 175.26 76.2 0)
 			(effects
@@
 		(on_board yes)
 		(dnp no)
-		(fields_autoplaced yes)
 		(property "Reference" "D1"
-			(at 142.24 22.86 0)
-			(effects
-				(font
-					(size 1.27 1.27)
-				)
-			)
-		)
-		(property "Value" "SMF5V0A"
-			(at 142.24 25.4 0)
+			(at 141.986 26.67 0)
+			(effects
+				(font
+					(size 1.27 1.27)
+				)
+			)
+		)
+		(property "Value" "ESD DIODE 5VWM 9.2VC"
+			(at 145.542 32.004 0)
 			(effects
 				(font
@@
 		)
 		(property "Description" "200W unidirectional Transil Transient Voltage Suppressor, 5Vrwm, SMF"
+			(at 142.24 29.21 0)
+			(effects
+				(font
+					(size 1.27 1.27)
+				)
+				(hide yes)
+			)
+		)
+		(property "MFR" "VISHAY"
+			(at 142.24 29.21 0)
+			(effects
+				(font
+					(size 1.27 1.27)
+				)
+				(hide yes)
+			)
+		)
+		(property "MPN" "SMF5V0A-E3-08"
+			(at 142.24 29.21 0)
+			(effects
+				(font
+					(size 1.27 1.27)
+				)
+				(hide yes)
+			)
+		)
+		(property "LCSPN" "C1972946"
 			(at 142.24 29.21 0)
 			(effects
@@
 			)
 		)
-		(property "Value" "5.6k"
+		(property "Value" "5.6kΩ ±1% 100mW"
 			(at 148.59 39.3699 0)
 			(effects
@@
 		)
 		(property "Description" "Resistor, small symbol"
+			(at 146.05 38.1 0)
+			(effects
+				(font
+					(size 1.27 1.27)
+				)
+				(hide yes)
+			)
+		)
+		(property "MFR" "FOJAN"
+			(at 146.05 38.1 0)
+			(effects
+				(font
+					(size 1.27 1.27)
+				)
+				(hide yes)
+			)
+		)
+		(property "MPN" "FRC0603F5601TS"
+			(at 146.05 38.1 0)
+			(effects
+				(font
+					(size 1.27 1.27)
+				)
+				(hide yes)
+			)
+		)
+		(property "LCSPN" "C2907046"
 			(at 146.05 38.1 0)
 			(effects
@@
 			)
 		)
-		(property "Value" "5.1k"
+		(property "Value" "5.1kΩ ±1% 100mW"
 			(at 140.97 55.88 90)
 			(effects
@@
 		(property "Description" "Resistor, small symbol"
 			(at 140.97 58.42 0)
+			(effects
+				(font
+					(size 1.27 1.27)
+				)
+				(hide yes)
+			)
+		)
+		(property "MFR" "FOJAN"
+			(at 140.97 58.42 90)
+			(effects
+				(font
+					(size 1.27 1.27)
+				)
+				(hide yes)
+			)
+		)
+		(property "MPN" "FRC0603F5101TS"
+			(at 140.97 58.42 90)
+			(effects
+				(font
+					(size 1.27 1.27)
+				)
+				(hide yes)
+			)
+		)
+		(property "LCSPN" "C2907044"
+			(at 140.97 58.42 90)
 			(effects
 				(font
@@
 			)
 		)
-		(property "Value" "10k"
+		(property "Value" "10kΩ ±1% 100mW"
 			(at 148.59 49.5299 0)
 			(effects
@@
 		)
 		(property "Description" "Resistor, small symbol"
+			(at 146.05 48.26 0)
+			(effects
+				(font
+					(size 1.27 1.27)
+				)
+				(hide yes)
+			)
+		)
+		(property "MFR" "UNI-ROYAL"
+			(at 146.05 48.26 0)
+			(effects
+				(font
+					(size 1.27 1.27)
+				)
+				(hide yes)
+			)
+		)
+		(property "MPN" "0603WAF1002T5E"
+			(at 146.05 48.26 0)
+			(effects
+				(font
+					(size 1.27 1.27)
+				)
+				(hide yes)
+			)
+		)
+		(property "LCSPN" "C25804"
 			(at 146.05 48.26 0)
 			(effects
@@
 			)
 		)
-		(property "Value" "5.1k"
+		(property "Value" "5.1kΩ ±1% 100mW"
 			(at 140.97 63.5 90)
 			(effects
@@
 			(effects
 				(font
+					(size 1.27 1.27)
+				)
+				(hide yes)
+			)
+		)
+		(property "MFR" "FOJAN"
+			(at 140.97 60.96 90)
+			(effects
+				(font
+					(size 1.27 1.27)
+				)
+				(hide yes)
+			)
+		)
+		(property "MPN" "FRC0603F5101TS"
+			(at 140.97 60.96 90)
+			(effects
+				(font
+					(size 1.27 1.27)
+				)
+				(hide yes)
+			)
+		)
+		(property "LCSPN" "C2907044"
+			(at 140.97 60.96 90)
+			(effects
+				(font
