File: hardware/hexaGenMini-v1/MCU.kicad_sch (KiCad schematic)
At the start: 25 parts, among them J3 Conn_01x03_Pin, SW1 TS-1088R-02026, SW2 TS-1088R-02026, U2 RP2040, U5 W25Q128JVS, Y1 12MHz 18pF

Commit message: Add base schematic for hardware
Parts:
- C10, C11, C12, C13, C14, C15, C16, C17, C5, C6, C9: footprint (none) -> Capacitor_SMD:C_0402_1005Metric
- C18, C7, C8, R5, R6, R7, R8, R9: footprint (none) -> Capacitor_SMD:C_0603_1608Metric
- J3: footprint (none) -> Connector_PinHeader_2.54mm:PinHeader_1x03_P2.54mm_Vertical
- SW1, SW2: value TS-1088R-02026 -> SW_Push; footprint (none) -> Button_Switch_SMD:SW_SPST_TL3342
- Y1: footprint (none) -> Crystal:Crystal_SMD_3215-2Pin_3.2x1.5mm
Connections:
- net at R9.1: now also SW2.2; no longer SW1.2
- net at U2.26 (RUN): now also SW1.2; no longer SW2.2
- net D+ renamed USB_DP
- net D- renamed USB_DM
- no-connect marks 0 -> 25

Commit message: Finish first hardware basic
Parts:
- added D2: WS2812B, LED_SMD:LED_WS2812B_PLCC4_5.0x5.0mm_P3.2mm, symbol SCH_Library:WS2812B
- added R19: 330, Resistor_SMD:R_0603_1608Metric, symbol SCH_Library:R_Small
- C10, C11, C12, C13, C14, C15, C16, C17, C18, C5, C6, C7, C8, C9: symbol Device:C_Small -> SCH_Library:C_Small
- J3: symbol Connector:Conn_01x03_Pin -> SCH_Library:Conn_01x03_Pin
- R5, R6, R7, R8, R9: footprint Capacitor_SMD:C_0603_1608Metric -> Resistor_SMD:R_0603_1608Metric; symbol Device:R_Small -> SCH_Library:R_Small
- SW1, SW2: footprint Button_Switch_SMD:SW_SPST_TL3342 -> Button_Switch_SMD:SW_SPST_B3U-1000P; symbol Switch:SW_Push -> SCH_Library:SW_Push
- U2: symbol MCU_RaspberryPi:RP2040 -> SCH_Library:RP2040
- U5: symbol Memory_Flash:W25Q128JVS -> SCH_Library:W25Q128JVS
- Y1: footprint Crystal:Crystal_SMD_3215-2Pin_3.2x1.5mm -> Crystal:Crystal_SMD_3225-4Pin_3.2x2.5mm; symbol Device:Crystal_GND24_Small -> SCH_Library:Crystal_GND24_Small
Connections:
- net GND: now also D2.3 (VSS)
- net SWCLK: now also J3.1 (Pin_1); no longer J3.3 (Pin_3)
- net SWD: now also J3.3 (Pin_3); no longer J3.1 (Pin_1)
- net RGB_LED: now reaches U2.8 (GPIO6)
- net RGB_LED: now also R19.1
- net USB_DM renamed USB_DN
- new net: D2.4 (DIN), R19.2
- new net +5V: D2.1 (VDD)

Commit message: Finish first hardware basic
Parts:
- C10, C11, C12, C13, C14, C15, C16, C17, C9: value 100nF -> CER 100nF 16V X7R; LCSPN (none) -> C1525; MFR (none) -> Samsung Electro-Mechanics; MPN (none) -> CL05B104KO5NNNC
- C18, C7, C8: value 1uF -> CER 1uF 50V X5R; LCSPN (none) -> C15849; MFR (none) -> Samsung Electro-Mechanics; MPN (none) -> CL10A105KB8NNNC
- C5, C6: value 27p -> CER 27pF 50V NP0; LCSPN (none) -> C107002; MFR (none) -> YAGEO; MPN (none) -> CC0402JRNPO9BN270
- D2: LCSPN (none) -> C2761795; MFR (none) -> Worldsemi; MPN (none) -> WS2812B-B/T
- J3: now left out of the parts list
- R19: value 330 -> 330Ω ±1% 100mW; LCSPN (none) -> C23138; MFR (none) -> UNI-ROYAL; MPN (none) -> 0603WAF3300T5E
- R5, R9: value 1k -> 1kΩ ±1% 100mW; LCSPN (none) -> C22548; MFR (none) -> YAGEO; MPN (none) -> RC0603FR-071KL
- R6, R7: value 27 -> 27Ω ±1% 100mW; LCSPN (none) -> C2907021; MFR (none) -> FOJAN; MPN (none) -> FRC0603F27R0TS
- R8: value 10k -> 10kΩ ±1% 100mW; LCSPN (none) -> C25804; MFR (none) -> UNI-ROYAL; MPN (none) -> 0603WAF1002T5E
- SW1, SW2: value SW_Push -> TACTILE SPST; LCSPN (none) -> C231329; MFR (none) -> OMRON; MPN (none) -> B3U-1000P
- U2: LCSPN (none) -> C2040; MFR (none) -> Raspberry Pi; MPN (none) -> RP2040
- U5: LCSPN (none) -> C97521; MFR (none) -> Winbond; MPN (none) -> W25Q128JVSIQ
- Y1: LCSPN (none) -> C91749; MFR (none) -> EPSON; MPN (none) -> Q22FA23V00418
